File: pcbs/acorn-system-1-gadget1/untitled.kicad_sch (KiCad schematic)
At the start: 2 parts

Commit message: "Update"
Connections:
- net GPIO10 renamed IRQ_DRV
- net GPIO16 renamed SD_SS
- net GPIO17 renamed SD_DAT2
- net GPIO18 renamed SD_DAT1
- net GPIO19 renamed MOSI_DI
- net GPIO20 renamed SD_CLK
- net GPIO22 renamed MISO_DO
- net GPIO8 renamed NRST_DRV
- net GPIO9 renamed NMI_DRV
Other:
- note added: "GPIO0-7 D0-D7"
- note added: "GPIO32-47 A0-A15"
- note removed: "EXTENSIONS"
- moved on the sheet: EXT1, EXT2
